File: Eagle Design/TeensyLED.brd (EAGLE design)
At the start: 50.8 x 80 mm, 68 parts, among them J1 22-05-7058-05, J2 PJ-202AH, Q1 ZXT1053AK, Q2 ZXT1053AK, Q3 ZXT1053AK, Q4 ZXT1053AK, U1 TEENSY_3.0_BASIC, U3 ADM2582E

Commit message: cleaned things up, testing readme.md inline images...
Parts:
- C13, C14, C15, C16: value 380pF -> 330pF
Changed lines of the file:
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@@
 <setting verticaltext="up"/>
 </settings>
-<grid distance="0.05" unitdist="inch" unit="inch" style="lines" multiple="1" display="no" altdistance="0.025" altunitdist="inch" altunit="inch"/>
+<grid distance="0.01" unitdist="inch" unit="inch" style="lines" multiple="1" display="no" altdistance="0.025" altunitdist="inch" altunit="inch"/>
 <layers>
-<layer number="1" name="Top" color="4" fill="1" visible="no" active="yes"/>
-<layer number="16" name="Bottom" color="1" fill="1" visible="no" active="yes"/>
-<layer number="17" name="Pads" color="2" fill="1" visible="no" active="yes"/>
-<layer number="18" name="Vias" color="2" fill="1" visible="no" active="yes"/>
+<layer number="1" name="Top" color="4" fill="1" visible="yes" active="yes"/>
+<layer number="16" name="Bottom" color="1" fill="1" visible="yes" active="yes"/>
+<layer number="17" name="Pads" color="2" fill="1" visible="yes" active="yes"/>
+<layer number="18" name="Vias" color="2" fill="1" visible="yes" active="yes"/>
 <layer number="19" name="Unrouted" color="6" fill="1" visible="yes" active="yes"/>
 <layer number="20" name="Dimension" color="15" fill="1" visible="yes" active="yes"/>
 <layer number="21" name="tPlace" color="7" fill="1" visible="yes" active="yes"/>
-<layer number="22" name="bPlace" color="7" fill="1" visible="no" active="yes"/>
-<layer number="23" name="tOrigins" color="15" fill="1" visible="no" active="yes"/>
-<layer number="24" name="bOrigins" color="15" fill="1" visible="no" active="yes"/>
+<layer number="22" name="bPlace" color="7" fill="1" visible="yes" active="yes"/>
+<layer number="23" name="tOrigins" color="15" fill="1" visible="yes" active="yes"/>
+<layer number="24" name="bOrigins" color="15" fill="1" visible="yes" active="yes"/>
 <layer number="25" name="tNames" color="7" fill="1" visible="yes" active="yes"/>
-<layer number="26" name="bNames" color="7" fill="1" visible="no" active="yes"/>
+<layer number="26" name="bNames" color="7" fill="1" visible="yes" active="yes"/>
 <layer number="27" name="tValues" color="7" fill="1" visible="no" active="yes"/>
 <layer number="28" name="bValues" color="7" fill="1" visible="no" active="yes"/>
@@
 <layer number="44" name="Drills" color="7" fill="1" visible="no" active="yes"/>
 <layer number="45" name="Holes" color="7" fill="1" visible="no" active="yes"/>
-<layer number="46" name="Milling" color="3" fill="1" visible="no" active="yes"/>
+<layer number="46" name="Milling" color="3" fill="1" visible="yes" active="yes"/>
 <layer number="47" name="Measures" color="7" fill="1" visible="yes" active="yes"/>
 <layer number="48" name="Document" color="7" fill="1" visible="yes" active="yes"/>
@@
 <attribute name="VALUE" x="30.226" y="42.545" size="1.27" layer="27" rot="R180"/>
 </element>
-<element name="C13" library="rcl" package="C0402PRO" value="380pF" x="29.083" y="39.116" smashed="yes">
+<element name="C13" library="rcl" package="C0402PRO" value="330pF" x="29.083" y="39.116" smashed="yes">
 <attribute name="NAME" x="30.48" y="38.608" size="1.016" layer="25"/>
 <attribute name="VALUE" x="28.575" y="38.735" size="1.016" layer="27" align="top-left"/>
@@
 <attribute name="VALUE" x="41.402" y="51.435" size="1.27" layer="27" rot="R180"/>
 </element>
-<element name="C14" library="rcl" package="C0402PRO" value="380pF" x="40.259" y="48.133" smashed="yes">
+<element name="C14" library="rcl" package="C0402PRO" value="330pF" x="40.259" y="48.133" smashed="yes">
 <attribute name="NAME" x="41.656" y="47.625" size="1.016" layer="25"/>
 <attribute name="VALUE" x="39.751" y="47.752" size="1.016" layer="27" align="top-left"/>
@@
 <attribute name="VALUE" x="40.132" y="13.335" size="1.27" layer="27" rot="R180"/>
 </element>
-<element name="C15" library="rcl" package="C0402PRO" value="380pF" x="38.989" y="10.033" smashed="yes">
+<element name="C15" library="rcl" package="C0402PRO" value="330pF" x="38.989" y="10.033" smashed="yes">
 <attribute name="NAME" x="40.386" y="9.525" size="1.016" layer="25"/>
 <attribute name="VALUE" x="38.481" y="9.652" size="1.016" layer="27" align="top-left"/>
@@
 <attribute name="VALUE" x="41.656" y="32.385" size="1.27" layer="27" rot="R180"/>
 </element>
-<element name="C16" library="rcl" package="C0402PRO" value="380pF" x="40.513" y="29.083" smashed="yes">
+<element name="C16" library="rcl" package="C0402PRO" value="330pF" x="40.513" y="29.083" smashed="yes">
 <attribute name="NAME" x="41.91" y="28.575" size="1.016" layer="25"/>
 <attribute name="VALUE" x="40.005" y="28.702" size="1.016" layer="27" align="top-left"/>
@@
 <via x="22.225" y="39.624" extent="1-16" drill="0.381"/>
 <contactref element="GND" pad="P$1"/>
+<via x="10.16" y="21.59" extent="1-16" drill="0.381"/>
+<via x="10.16" y="20.574" extent="1-16" drill="0.381"/>
+<via x="10.16" y="19.558" extent="1-16" drill="0.381"/>
+<via x="10.16" y="18.542" extent="1-16" drill="0.381"/>
+<via x="11.176" y="18.542" extent="1-16" drill="0.381"/>
+<via x="11.176" y="19.558" extent="1-16" drill="0.381"/>
+<via x="11.176" y="20.574" extent="1-16" drill="0.381"/>
+<via x="11.176" y="21.59" extent="1-16" drill="0.381"/>
 </signal>
 <signal name="VCC">
