File: Eagle Design/TeensyLED.sch (EAGLE design)
At the start: 68 parts, among them J1 22-05-7058-05, J2 PJ-202AH, Q1 ZXT1053AK, Q2 ZXT1053AK, Q3 ZXT1053AK, Q4 ZXT1053AK, U1 TEENSY_3.0_BASIC, U2 LMR16006YDDCT, U3 ADM2582E

Commit message: cleaned things up, testing readme.md inline images...
Parts:
- C13, C14, C15, C16: value 380pF -> 330pF
Other:
- moved on the sheet: C10, C11, C12, C5, C6, C7, C8, C9, GISO, U3, VISO
